File: inzynierka/inzynierka.kicad_pcb (KiCad board)
At the start: 2 copper layers, 95.8 x 52 mm, 107 parts, among them J101 Conn_01x10, Q501 Q_PNP_BCE, Q502 BC848, T501 Transformer_1P_1S, U101 LM1117-3.3, U102 MCP6L04x-xSL, U103 LM239D, U201 SPU0410LR5H-QB, U202 MCP6L04x-xSL, U301 SPU0410LR5H-QB, U302 MCP6L04x-xSL, U401 SPU0410LR5H-QB, U402 MCP6L04x-xSL

Commit message: shield shape
Parts:
- added C501: C_Small, Capacitor_SMD:C_0603_1608Metric, F.Cu at (124.8, 86.5)
- added D503: 1N5819WS, Diode_SMD:D_SOD-323, F.Cu at (126.4, 90.0)
- added H101: MountingHole, MountingHole:MountingHole_3.2mm_M3, F.Cu at (114.9, 134.5)
- added H102: MountingHole, MountingHole:MountingHole_3.2mm_M3, F.Cu at (87.0, 134.5)
- added H103: MountingHole, MountingHole:MountingHole_3.2mm_M3, F.Cu at (130.1, 83.7)
- added H104: MountingHole, MountingHole:MountingHole_3.2mm_M3, F.Cu at (81.9, 82.4)
- added H501: BuzzerHole, MountingHole:MountingHole_2.2mm_M2, F.Cu at (92.8, 63.9)
- added J102: SHIELD_RIGHT, Connector_PinSocket_2.54mm:PinSocket_2x19_P2.54mm_Vertical, B.Cu at (135.2, 86.2)
- BZ501: footprint Buzzer_Beeper:Buzzer_12x9.5RM7.6 -> Buzzer_Beeper:Buzzer_15x7.5RM7.6
- D501: value US1M -> 1N5819WS; footprint Diode_SMD:D_SMA -> Diode_SMD:D_SOD-323
- J101: value Conn_01x10 -> SHIELD_LEFT; footprint Connector_JST:JST_XH_B10B-XH-A_1x10_P2.50mm_Vertical -> Connector_PinSocket_2.54mm:PinSocket_2x19_P2.54mm_Vertical; moved to B.Cu
- Q501: value Q_PNP_BCE -> SS8550
- Q502: value BC848 -> MMBT3904
- moved J101 155.2 mm to (74.2, 86.2), turned to 180 degrees
- moved C108 136.9 mm to (88.2, 93.9), turned to 180 degrees
- moved R106 136.1 mm to (88.2, 95.4), turned to 180 degrees
- moved C101 134.3 mm to (90.2, 84.4), turned to 90 degrees
- moved TP202 133.5 mm to (81.2, 123.0), turned to 90 degrees
- moved C202 133.1 mm to (81.8, 119.8), turned to 90 degrees
- moved R104 133.1 mm to (91.2, 93.9), turned to 0 degrees
- moved R105 132.2 mm to (91.2, 95.4), turned to 180 degrees
- moved C105 130.0 mm to (85.7, 102.0)
- moved C102 129.6 mm to (93.5, 86.1), turned to 90 degrees
- moved R202 129.1 mm to (84.2, 124.8), turned to 0 degrees
- moved C205 129.1 mm to (84.2, 126.2), turned to 0 degrees
- moved C203 129.1 mm to (84.2, 129.2), turned to 0 degrees
- moved C210 129.1 mm to (85.2, 114.8), turned to 180 degrees
- moved R201 129.0 mm to (84.2, 127.8), turned to 180 degrees
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Connections:
- BZ501 pad 1: Net-(BZ501-Pad1) -> Net-(T501-Pad1)
- BZ501 pad 2: Net-(BZ501-Pad2) -> Net-(T501-Pad2)
- C105 pad 2: GND -> GNDA
- C107 pad 2: GND -> GNDA
- C108 pad 2: GND -> GNDA
- C201 pad 2: GND -> GNDA
- C202 pad 2: GND -> GNDA
- C204 pad 1: GND -> GNDA
- C210 pad 2: GND -> GNDA
- C301 pad 2: GND -> GNDA
- C302 pad 2: GND -> GNDA
- C304 pad 1: GND -> GNDA
- C310 pad 2: GND -> GNDA
- C401 pad 2: GND -> GNDA
- C402 pad 2: GND -> GNDA
- C404 pad 1: GND -> GNDA
- C410 pad 2: GND -> GNDA
- D501 pad 1: Net-(D501-Pad1) -> Net-(Q501-Pad3)
- J101 pad 1: +5V -> unconnected-(J101-Pad1)
- J101 pad 2: +3V3 -> unconnected-(J101-Pad2)
- J101 pad 3: GND -> unconnected-(J101-Pad3)
- J101 pad 4: OUT_0 -> unconnected-(J101-Pad4)
- J101 pad 5: OUT_1 -> unconnected-(J101-Pad5)
- J101 pad 6: OUT_2 -> unconnected-(J101-Pad6)
- J101 pad 7: PIEZO -> unconnected-(J101-Pad7)
- J101 pad 8: THRESHOLD_MCU -> GND
- J101 pad 9: AREF -> unconnected-(J101-Pad9)
- Q501 pad 2: Net-(D501-Pad1) -> +5V
- Q501 pad 3: +3V3 -> Net-(Q501-Pad3)
- R104 pad 2: GND -> GNDA
- R106 pad 2: GND -> GNDA
- R502 pad 2: PIEZO -> Net-(R502-Pad2)
- R503 pad 1: Net-(D501-Pad1) -> Net-(Q501-Pad3)
- T501 pad 1: Net-(BZ501-Pad2) -> Net-(T501-Pad1)
- T501 pad 2: Net-(BZ501-Pad1) -> Net-(T501-Pad2)
- T501 pad 4: Net-(D501-Pad1) -> Net-(Q501-Pad3)
- TP501 pad 1: Net-(D501-Pad1) -> Net-(Q501-Pad3)
- TP502 pad 1: PIEZO -> /TRANSMITER/PIEZO_IN
- U102 pad 11: GND -> GNDA
- U201 pad 2: GND -> GNDA
- U201 pad 3: GND -> GNDA
- U201 pad 5: GND -> GNDA
- U201 pad 6: GND -> GNDA
- U202 pad 11: GND -> GNDA
- U301 pad 2: GND -> GNDA
- U301 pad 3: GND -> GNDA
- U301 pad 5: GND -> GNDA
- U301 pad 6: GND -> GNDA
- U302 pad 11: GND -> GNDA
- U401 pad 2: GND -> GNDA
- U401 pad 3: GND -> GNDA
- U401 pad 5: GND -> GNDA
- U401 pad 6: GND -> GNDA
- U402 pad 11: GND -> GNDA
Routing:
- net +3V3: track 11.1 -> 164.1 mm, vias 0 -> 13
- net THRESHOLD_MCU: track 10.4 -> 54.4 mm
- net OUT_2: track 5.02 -> 42.7 mm, vias 0 -> 1
- net OUT_0: track 4.95 -> 41.3 mm, vias 0 -> 1
- net OUT_1: track 5.02 -> 38.9 mm, vias 0 -> 1
- net MIC_0: track 4.05 -> 31.0 mm
- net MIC_2: track 4.05 -> 29.2 mm
- net THRESHOLD_OP: track 1.27 -> 14.9 mm
- net MIC_1: track 4.05 -> 16.1 mm
- net Net-(C305-Pad2): track 10.9 -> 18.7 mm
Other:
- board size 95.8 x 52 mm -> 69.6 x 95.5 mm
- board text removed: "NC AREF THOLD BUZZER MIC_2 MIC_1 MIC_0 GND 3V3 5V"

Commit message: skonczone pcb
Parts:
- removed BZ501: Buzzer, Buzzer_Beeper:Buzzer_15x7.5RM7.6
- removed H501: BuzzerHole, MountingHole:MountingHole_2.2mm_M2
- added BZ101: Buzzer, Buzzer_Beeper:Buzzer_15x7.5RM7.6, F.Cu at (118.7, 70.5)
- added C112: 100n, Capacitor_SMD:C_0603_1608Metric, F.Cu at (81.2, 96.5)
- added D104: DBG, LED_SMD:LED_0603_1608Metric, F.Cu at (123.3, 82.7)
- added H105: BuzzerHole, MountingHole:MountingHole_2.2mm_M2, F.Cu at (92.8, 64.0)
- added J104: PIEZO, Connector_PinHeader_2.54mm:PinHeader_1x02_P2.54mm_Vertical, F.Cu at (128.9, 132.7)
- added J105: FPC, Connector_FFC-FPC:Hirose_FH12-10S-0.5SH_1x10-1MP_P0.50mm_Horizontal, F.Cu at (105.6, 65.7)
- added J106: FPC, Connector_FFC-FPC:Hirose_FH12-10S-0.5SH_1x10-1MP_P0.50mm_Horizontal, F.Cu at (96.1, 134.6)
- added R110: 1k, Resistor_SMD:R_0603_1608Metric, F.Cu at (121.8, 82.7)
- added R111: 1k, Resistor_SMD:R_0603_1608Metric, F.Cu at (81.2, 93.5)
- added R112: 10k, Resistor_SMD:R_0603_1608Metric, F.Cu at (81.2, 90.5)
- added SW101: DBG, Button_Switch_SMD:SW_SPST_B3S-1000, F.Cu at (87.5, 93.0)
- added TP107: B+, TestPoint:TestPoint_Pad_D2.0mm, F.Cu at (119.0, 74.6)
- added TP108: B-, TestPoint:TestPoint_Pad_D2.0mm, F.Cu at (126.1, 74.6)
- added kibuzzard-636196D3: G***, kibuzzard-636196D3, F.Cu at (84.5, 52.5)
- added kibuzzard-636196F7: G***, kibuzzard-636196F7, F.Cu at (89.2, 52.5)
- added kibuzzard-636196FE: G***, kibuzzard-636196FE, F.Cu at (89.2, 54.8)
- added kibuzzard-6361BCC4: G***, kibuzzard-6361BCC4, B.Cu at (106.0, 124.9)
- added kibuzzard-6361BD58: G***, kibuzzard-6361BD58, F.Cu at (125.1, 82.7)
- added kibuzzard-6361BD6E: G***, kibuzzard-6361BD6E, F.Cu at (115.1, 82.7)
- added kibuzzard-6361BD82: G***, kibuzzard-6361BD82, F.Cu at (120.1, 82.7)
- added kibuzzard-6361C7A3: G***, kibuzzard-6361C7A3, F.Cu at (95.3, 95.9)
- added kibuzzard-6361C7DF: G***, kibuzzard-6361C7DF, F.Cu at (113.1, 93.6)
- added mouse-bite-2mm-slot: VAL**, Panelization:mouse-bite-2mm-slot, F.Cu at (116.2, 59.9)
- added mouse-bite-2mm-slot: VAL**, Panelization:mouse-bite-2mm-slot, F.Cu at (122.5, 62.1)
- added mouse-bite-2mm-slot: VAL**, Panelization:mouse-bite-2mm-slot, F.Cu at (97.1, 78.9)
- added mouse-bite-2mm-slot: VAL**, Panelization:mouse-bite-2mm-slot, F.Cu at (122.5, 78.9)
- T501: value Transformer_1P_1S -> Transformer_Audio; footprint Transformer_THT:Transformer_Toroid_Horizontal_D9.0mm_Amidon-T30 -> Transformer:Transformer_shielded_8x13.5
- TP101, TP106: value TestPoint -> THR
- TP102, TP204, TP304, TP404: value TestPoint -> OP
- TP103: value TestPoint -> OUT_0
- TP104: value TestPoint -> OUT_1
- TP105: value TestPoint -> OUT_2
- TP201, TP301, TP401: value TestPoint -> M_AC
- TP202, TP302, TP402: value TestPoint -> 1STG
- TP203, TP303, TP403: value TestPoint -> 2STG
- TP501, TP502: value TestPoint -> P
- moved D103 16.9 mm to (97.2, 96.0), turned to -90 degrees
- moved R503 15.7 mm to (113.4, 90.3), turned to 0 degrees
- moved R109 15.3 mm to (98.7, 96.0), turned to 90 degrees
- moved TP502 13.8 mm to (132.4, 95.5)
- moved D502 13.6 mm to (113.4, 91.8), turned to 180 degrees
- moved C105 12.2 mm to (97.8, 104.0), turned to -90 degrees
- moved C108 11.9 mm to (84.0, 105.0), turned to -90 degrees
- moved R104 10.8 mm to (84.0, 102.0), turned to 90 degrees
- moved C501 10.0 mm to (132.5, 92.9), turned to 90 degrees
- moved R106 9.96 mm to (85.5, 105.0), turned to -90 degrees
- moved R502 9.11 mm to (128.1, 92.8), turned to 90 degrees
- moved TP501 9.07 mm to (113.8, 96.2)
- moved Q501 8.93 mm to (117.9, 93.6), turned to 180 degrees
- moved R105 8.72 mm to (85.5, 102.0), turned to -90 degrees
- moved R501 7.48 mm to (121.5, 93.6)
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Connections:
- C105 pad 2: GNDA -> GND
- C107 pad 2: GNDA -> GND
- C108 pad 2: GNDA -> GND
- C201 pad 2: GNDA -> GND
- C202 pad 2: GNDA -> GND
- C203 pad 1: Net-(C203-Pad1) -> /MIC_0/MIC_RAW
- C204 pad 1: GNDA -> GND
- C210 pad 2: GNDA -> GND
- C301 pad 2: GNDA -> GND
- C302 pad 2: GNDA -> GND
- C303 pad 1: Net-(C303-Pad1) -> /MIC_1/MIC_RAW
- C304 pad 1: GNDA -> GND
- C310 pad 2: GNDA -> GND
- C401 pad 2: GNDA -> GND
- C402 pad 2: GNDA -> GND
- C403 pad 1: Net-(C403-Pad1) -> /MIC_2/MIC_RAW
- C404 pad 1: GNDA -> GND
- C410 pad 2: GNDA -> GND
- C501 pad 2: /TRANSMITER/PIEZO_IN -> PIEZO
- J101 pad 2: unconnected-(J101-Pad2) -> DBG_BUT
- J101 pad 34: PIEZO -> unconnected-(J101-Pad34)
- J102 pad 1: unconnected-(J102-Pad1) -> DBG_LED
- J102 pad 13: unconnected-(J102-Pad13) -> PIEZO
- R104 pad 2: GNDA -> GND
- R106 pad 2: GNDA -> GND
- T501 pad 1: Net-(T501-Pad1) -> /TRANSMITER/BUZZER+
- T501 pad 2: Net-(T501-Pad2) -> /TRANSMITER/BUZZER-
- TP502 pad 1: /TRANSMITER/PIEZO_IN -> PIEZO
- U102 pad 11: GNDA -> GND
- U201 pad 1: Net-(C203-Pad1) -> Net-(J105-Pad5)
- U201 pad 2: GNDA -> GND
- U201 pad 3: GNDA -> GND
- U201 pad 5: GNDA -> GND
- U201 pad 6: GNDA -> GND
- U202 pad 11: GNDA -> GND
- U301 pad 1: Net-(C303-Pad1) -> Net-(J105-Pad3)
- U301 pad 2: GNDA -> GND
- U301 pad 3: GNDA -> GND
- U301 pad 5: GNDA -> GND
- U301 pad 6: GNDA -> GND
- U302 pad 11: GNDA -> GND
- U401 pad 1: Net-(C403-Pad1) -> Net-(J105-Pad7)
- U401 pad 2: GNDA -> GND
- U401 pad 3: GNDA -> GND
- U401 pad 5: GNDA -> GND
- U401 pad 6: GNDA -> GND
- U402 pad 11: GNDA -> GND
Routing:
- net +3V3: track 164.1 -> 260.2 mm
- net GND: track 0.00 -> 89.4 mm, vias 0 -> 16
- net +5V: track 8.96 -> 81.9 mm, vias 0 -> 3
- net OPERATING_POINT: track 17.0 -> 70.7 mm, vias 0 -> 5
- net /TRANSMITER/BUZZER-: track 0.00 -> 34.1 mm
- net THRESHOLD_OP: track 14.9 -> 44.7 mm, vias 0 -> 3
- net /TRANSMITER/BUZZER+: track 0.00 -> 27.1 mm
- net Net-(J105-Pad5): track 0.00 -> 27.1 mm
- net Net-(D501-Pad1): track 0.00 -> 27.1 mm
- net /MIC_2/MIC_RAW: track 0.00 -> 23.6 mm
- net Net-(J105-Pad3): track 0.00 -> 19.2 mm
- net DBG_LED: track 0.00 -> 16.0 mm
- net Net-(J105-Pad7): track 0.00 -> 15.9 mm
- net Net-(C112-Pad1): track 0.00 -> 13.9 mm
- net /MIC_0/MIC_RAW: track 0.00 -> 12.7 mm
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Other:
- board size 69.6 x 95.5 mm -> 69.6 x 95.6 mm
- board text added: "JLCJLCJLCJLC"
- board text removed: "5mm"
