File: inzynierka/MIC_0.kicad_sch (KiCad schematic)
At the start: 22 parts, among them U201 SPU0410LR5H-QB, U202 MCP6L04x-xSL

Commit message: skonczone pcb
Parts:
- removed C201: 100n, Capacitor_SMD:C_0603_1608Metric, symbol Device:C_Small
- removed U201: SPU0410LR5H-QB, SPU0410:SPU0410LR5H-QB, symbol SPU0410LR5H-QB:SPU0410LR5H-QB
- TP201: value TestPoint -> M_AC
- TP202: value TestPoint -> 1STG
- TP203: value TestPoint -> 2STG
- TP204: value TestPoint -> OP
Connections:
- net MIC_RAW: now reaches C203.1
- net GNDA renamed GND
- net MIC_0 renamed MIC
Other:
- note removed: "Microphone"
- company: (none) -> Krystian Mirek
- title: (none) -> UltraSoundSensor

Commit message: production files
Parts:
- C203, C206, C208: value C_Small -> 2n
- C205, C207: value C_Small -> 117p
- C209: value C_Small -> 39p
- R202: value R_Small -> 25.5k
- R204: value R_Small -> 51k
- R205: value R_Small -> 500R
- R206: value R_Small -> 100k
Changed lines of the file:
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@@
     (in_bom yes) (on_board yes) (fields_autoplaced)
     (property "Reference" "C206" (id 0) (at 124.4663 44.45 90))
-    (property "Value" "C_Small" (id 1) (at 124.4663 46.99 90))
+    (property "Value" "2n" (id 1) (at 124.4663 46.99 90))
     (property "Footprint" "Capacitor_SMD:C_0603_1608Metric" (id 2) (at 124.46 50.8 0)
       (effects (font (size 1.27 1.27)) hide)
@@
     (in_bom yes) (on_board yes) (fields_autoplaced)
     (property "Reference" "R205" (id 0) (at 187.96 44.45 90))
-    (property "Value" "R_Small" (id 1) (at 187.96 46.99 90))
+    (property "Value" "500R" (id 1) (at 187.96 46.99 90))
     (property "Footprint" "Resistor_SMD:R_0603_1608Metric" (id 2) (at 187.96 50.8 0)
       (effects (font (size 1.27 1.27)) hide)
@@
     (in_bom yes) (on_board yes)
     (property "Reference" "C203" (id 0) (at 58.4263 44.45 90))
-    (property "Value" "C_Small" (id 1) (at 58.4263 46.99 90))
+    (property "Value" "2n" (id 1) (at 58.4263 46.99 90))
     (property "Footprint" "Capacitor_SMD:C_0603_1608Metric" (id 2) (at 58.42 50.8 0)
       (effects (font (size 1.27 1.27)) hide)
@@
     (in_bom yes) (on_board yes) (fields_autoplaced)
     (property "Reference" "C208" (id 0) (at 177.8063 44.45 90))
-    (property "Value" "C_Small" (id 1) (at 177.8063 46.99 90))
+    (property "Value" "2n" (id 1) (at 177.8063 46.99 90))
     (property "Footprint" "Capacitor_SMD:C_0603_1608Metric" (id 2) (at 177.8 50.8 0)
       (effects (font (size 1.27 1.27)) hide)
@@
     (in_bom yes) (on_board yes) (fields_autoplaced)
     (property "Reference" "C205" (id 0) (at 96.5263 24.13 90))
-    (property "Value" "C_Small" (id 1) (at 96.5263 26.67 90))
+    (property "Value" "117p" (id 1) (at 96.5263 26.67 90))
     (property "Footprint" "Capacitor_SMD:C_0603_1608Metric" (id 2) (at 96.52 30.48 0)
       (effects (font (size 1.27 1.27)) hide)
@@
     (in_bom yes) (on_board yes) (fields_autoplaced)
     (property "Reference" "R202" (id 0) (at 96.52 34.29 90))
-    (property "Value" "R_Small" (id 1) (at 96.52 36.83 90))
+    (property "Value" "25.5k" (id 1) (at 96.52 36.83 90))
     (property "Footprint" "Resistor_SMD:R_0603_1608Metric" (id 2) (at 96.52 40.64 0)
       (effects (font (size 1.27 1.27)) hide)
@@
     (in_bom yes) (on_board yes) (fields_autoplaced)
     (property "Reference" "C209" (id 0) (at 203.2063 24.13 90))
-    (property "Value" "C_Small" (id 1) (at 203.2063 26.67 90))
+    (property "Value" "39p" (id 1) (at 203.2063 26.67 90))
     (property "Footprint" "Capacitor_SMD:C_0603_1608Metric" (id 2) (at 203.2 30.48 0)
       (effects (font (size 1.27 1.27)) hide)
@@
     (in_bom yes) (on_board yes) (fields_autoplaced)
     (property "Reference" "R204" (id 0) (at 149.86 34.29 90))
-    (property "Value" "R_Small" (id 1) (at 149.86 36.83 90))
+    (property "Value" "51k" (id 1) (at 149.86 36.83 90))
     (property "Footprint" "Resistor_SMD:R_0603_1608Metric" (id 2) (at 149.86 40.64 0)
       (effects (font (size 1.27 1.27)) hide)
@@
     (in_bom yes) (on_board yes) (fields_autoplaced)
     (property "Reference" "R206" (id 0) (at 203.2 34.29 90))
-    (property "Value" "R_Small" (id 1) (at 203.2 36.83 90))
+    (property "Value" "100k" (id 1) (at 203.2 36.83 90))
     (property "Footprint" "Resistor_SMD:R_0603_1608Metric" (id 2) (at 203.2 40.64 0)
       (effects (font (size 1.27 1.27)) hide)
@@
     (in_bom yes) (on_board yes) (fields_autoplaced)
     (property "Reference" "C207" (id 0) (at 149.8663 24.13 90))
-    (property "Value" "C_Small" (id 1) (at 149.8663 26.67 90))
+    (property "Value" "117p" (id 1) (at 149.8663 26.67 90))
     (property "Footprint" "Capacitor_SMD:C_0603_1608Metric" (id 2) (at 149.86 30.48 0)
       (effects (font (size 1.27 1.27)) hide)
