File: inzynierka/transmiter.kicad_sch (KiCad schematic)
At the start: 11 parts, among them Q501 Q_PNP_BCE, Q502 BC848, T501 Transformer_1P_1S

Commit message: shield shape
Parts:
- removed D501: US1M, Diode_SMD:D_SMA, symbol Diode:US1M
- removed Q501: Q_PNP_BCE, Package_TO_SOT_SMD:SOT-23, symbol Device:Q_PNP_BCE
- removed Q502: BC848, Package_TO_SOT_SMD:SOT-23, symbol Transistor_BJT:BC848
- added C501: C_Small, Capacitor_SMD:C_0603_1608Metric, symbol Device:C_Small
- added D501, D503: 1N5819WS, Diode_SMD:D_SOD-323, symbol Diode:1N5819WS
- added H501: BuzzerHole, MountingHole:MountingHole_2.2mm_M2, symbol Mechanical:MountingHole
- added Q501: SS8550, Package_TO_SOT_SMD:SOT-23, symbol Device:Q_PNP_BEC
- added Q502: MMBT3904, Package_TO_SOT_SMD:SOT-23, symbol Transistor_BJT:MMBT3904
- BZ501: footprint Buzzer_Beeper:Buzzer_12x9.5RM7.6 -> Buzzer_Beeper:Buzzer_15x7.5RM7.6
Connections:
- net GND: now also D501.2 (A), D503.2 (A), Q502.2 (E)
- net at R501.1: now also Q502.3 (C)
- net at R501.2: now also Q501.1 (B)
- net at R502.1: now also Q502.1 (B)
- net at R503.1, T501.4 (SB), TP501.1: now also D501.1 (K), Q501.3 (C)
- net at T501.1 (AA): now also BZ501.1 (-); no longer BZ501.2 (+)
- net at T501.2 (AB): now also BZ501.2 (+); no longer BZ501.1 (-)
- net PIEZO: no longer names the net of R502.2
- net PIEZO: now also C501.1, D503.1 (K); no longer TP502.1
- new net +5V: Q501.2 (E)
- new net PIEZO_IN: C501.2, TP502.1
Other:
- moved on the sheet: D502, R501, R502, R503, T501, TP501

Commit message: skonczone pcb
Parts:
- removed BZ501: Buzzer, Buzzer_Beeper:Buzzer_15x7.5RM7.6, symbol Device:Buzzer
- removed H501: BuzzerHole, MountingHole:MountingHole_2.2mm_M2, symbol Mechanical:MountingHole
- removed T501: Transformer_1P_1S, Transformer_THT:Transformer_Toroid_Horizontal_D9.0mm_Amidon-T30, symbol Device:Transformer_1P_1S
- added T501: Transformer_Audio, Transformer:Transformer_shielded_8x13.5, symbol Device:Transformer_Audio
- TP501, TP502: value TestPoint -> P
Connections:
- net GND: now also T501.0, T501.3 (SA)
- net at D501.1 (K), Q501.3 (C), R503.1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: now also T501.4 (SB)
- net PIEZO_IN renamed INPUT
- new net BUZZER+: T501.1 (AA)
- new net BUZZER-: T501.2 (AB)
Other:
- company: (none) -> Krystian Mirek
- title: (none) -> UltraSoundSensor
Changed lines of the file:
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@@
 (kicad_sch (version 20211123) (generator eeschema)
   (paper "User" 150.012 99.9998)
+  (title_block
+    (title "UltraSoundSensor")
+    (date "2022-10-30")
+    (rev "1.0")
+    (company "Krystian Mirek")
+  )
   (junction (at 60.96 43.18) (diameter 0) (color 0 0 0 0)
   )
@@
   (junction (at 54.61 33.02) (diameter 0) (color 0 0 0 0)
   )
+  (wire (pts (xy 41.91 48.26) (xy 41.91 49.53))
+    (stroke (width 0) (type default) (color 0 0 0 0))
+  )
   (wire (pts (xy 71.12 34.29) (xy 71.12 33.02))
     (stroke (width 0) (type default) (color 0 0 0 0))
@@
     (stroke (width 0) (type default) (color 0 0 0 0))
   )
-  (wire (pts (xy 25.4 40.64) (xy 25.4 43.18))
-    (stroke (width 0) (type default) (color 0 0 0 0))
-  )
   (wire (pts (xy 107.95 39.37) (xy 107.95 40.64))
     (stroke (width 0) (type default) (color 0 0 0 0))
@@
     (stroke (width 0) (type default) (color 0 0 0 0))
   )
-  (wire (pts (xy 25.4 35.56) (xy 25.4 33.02))
-    (stroke (width 0) (type default) (color 0 0 0 0))
-  )
   (wire (pts (xy 91.44 33.02) (xy 91.44 34.29))
     (stroke (width 0) (type default) (color 0 0 0 0))
@@
     (stroke (width 0) (type default) (color 0 0 0 0))
   )
-  (wire (pts (xy 21.59 35.56) (xy 25.4 35.56))
-    (stroke (width 0) (type default) (color 0 0 0 0))
-  )
   (wire (pts (xy 60.96 33.02) (xy 60.96 34.29))
     (stroke (width 0) (type default) (color 0 0 0 0))
@@
     (stroke (width 0) (type default) (color 0 0 0 0))
   )
-  (wire (pts (xy 21.59 40.64) (xy 25.4 40.64))
-    (stroke (width 0) (type default) (color 0 0 0 0))
-  )
   (wire (pts (xy 60.96 43.18) (xy 60.96 41.91))
     (stroke (width 0) (type default) (color 0 0 0 0))
@@
     (stroke (width 0) (type default) (color 0 0 0 0))
   )
-  (hierarchical_label "PIEZO_IN" (shape input) (at 125.73 39.37 0)
+  (hierarchical_label "BUZZER+" (shape input) (at 25.4 33.02 180)
+    (effects (font (size 1.27 1.27) bold) (justify right))
+  )
+  (hierarchical_label "INPUT" (shape input) (at 125.73 39.37 0)
     (effects (font (size 1.27 1.27)) (justify left))
+  )
+  (hierarchical_label "BUZZER-" (shape input) (at 25.4 43.18 180)
+    (effects (font (size 1.27 1.27) bold) (justify right))
   )
   (symbol (lib_id "power:GND") (at 107.95 49.53 0) (unit 1)
@@
     (pin "1")
     (pin "2")
-  )
-  (symbol (lib_id "Mechanical:MountingHole") (at 20.32 52.07 0) (unit 1)
-    (in_bom yes) (on_board yes) (fields_autoplaced)
-    (property "Reference" "H501" (id 0) (at 22.86 50.7999 0)
-      (effects (font (size 1.27 1.27)) (justify left))
-    )
-    (property "Value" "BuzzerHole" (id 1) (at 22.86 53.3399 0)
-      (effects (font (size 1.27 1.27)) (justify left))
-    )
-    (property "Footprint" "MountingHole:MountingHole_2.2mm_M2" (id 2) (at 20.32 52.07 0)
-      (effects (font (size 1.27 1.27)) hide)
-    )
-    (property "Datasheet" "~" (id 3) (at 20.32 52.07 0)
-      (effects (font (size 1.27 1.27)) hide)
-    )
   )
   (symbol (lib_id "Device:R_Small") (at 102.87 39.37 90) (unit 1)
@@
     (pin "1")
   )
+  (symbol (lib_id "Device:Transformer_Audio") (at 41.91 38.1 0) (unit 1)
+    (in_bom yes) (on_board yes) (fields_autoplaced)
+    (property "Reference" "T501" (id 0) (at 41.91 25.4 0))
+    (property "Value" "Transformer_Audio" (id 1) (at 41.91 27.94 0))
+    (property "Footprint" "Transformer:Transformer_shielded_8x13.5" (id 2) (at 41.91 38.1 0)
+      (effects (font (size 1.27 1.27)) hide)
+    )
+    (property "Datasheet" "~" (id 3) (at 41.91 38.1 0)
+      (effects (font (size 1.27 1.27)) hide)
+    )
+    (pin "0")
+    (pin "1")
+    (pin "2")
+    (pin "3")
+    (pin "4")
+  )
   (symbol (lib_id "Connector:TestPoint") (at 54.61 30.48 0) (unit 1)
     (in_bom yes) (on_board yes)
@@
       (effects (font (size 1.27 1.27)) (justify left))
     )
-    (property "Value" "TestPoint" (id 1) (at 54.61 25.4 90)
+    (property "Value" "P" (id 1) (at 54.61 25.4 90)
       (effects (font (size 1.27 1.27)) (justify left))
     )
@@
     (pin "2")
     (pin "3")
-  )
-  (symbol (lib_id "Device:Buzzer") (at 19.05 38.1 0) (mirror y) (unit 1)
-    (in_bom yes) (on_board yes) (fields_autoplaced)
-    (property "Reference" "BZ501" (id 0) (at 18.288 29.21 0))
-    (property "Value" "Buzzer" (id 1) (at 18.288 31.75 0))
-    (property "Footprint" "Buzzer_Beeper:Buzzer_15x7.5RM7.6" (id 2) (at 19.685 35.56 90)
-      (effects (font (size 1.27 1.27)) hide)
-    )
-    (property "Datasheet" "~" (id 3) (at 19.685 35.56 90)
-      (effects (font (size 1.27 1.27)) hide)
-    )
-    (pin "1")
-    (pin "2")
   )
   (symbol (lib_id "Device:Q_PNP_BEC") (at 63.5 26.67 180) (unit 1)
@@
     (pin "3")
   )
-  (symbol (lib_id "Device:Transformer_1P_1S") (at 41.91 38.1 0) (unit 1)
-    (in_bom yes) (on_board yes) (fields_autoplaced)
-    (property "Reference" "T501" (id 0) (at 41.9227 27.94 0))
-    (property "Value" "Transformer_1P_1S" (id 1) (at 41.9227 30.48 0))
-    (property "Footprint" "Transformer_THT:Transformer_Toroid_Horizontal_D9.0mm_Amidon-T30" (id 2) (at 41.91 38.1 0)
-      (effects (font (size 1.27 1.27)) hide)
-    )
-    (property "Datasheet" "~" (id 3) (at 41.91 38.1 0)
-      (effects (font (size 1.27 1.27)) hide)
-    )
-    (pin "1")
-    (pin "2")
-    (pin "3")
-    (pin "4")
-  )
   (symbol (lib_id "Device:R_Small") (at 71.12 36.83 0) (unit 1)
     (in_bom yes) (on_board yes) (fields_autoplaced)
@@
       (effects (font (size 1.27 1.27)) (justify left))
     )
-    (property "Value" "TestPoint" (id 1) (at 123.19 33.02 90)
+    (property "Value" "P" (id 1) (at 123.19 33.02 90)
       (effects (font (size 1.27 1.27)) (justify left))
     )
@@
       (effects (font (size 1.27 1.27)) hide)
     )
+    (pin "1")
+  )
+  (symbol (lib_id "power:GND") (at 41.91 49.53 0) (unit 1)
+    (in_bom yes) (on_board yes) (fields_autoplaced)
+    (property "Reference" "#PWR0164" (id 0) (at 41.91 55.88 0)
+      (effects (font (size 1.27 1.27)) hide)
+    )
+    (property "Value" "GND" (id 1) (at 41.91 54.61 0))
+    (property "Footprint" "" (id 2) (at 41.91 49.53 0)
+      (effects (font (size 1.27 1.27)) hide)
+    )
+    (property "Datasheet" "" (id 3) (at 41.91 49.53 0)
+      (effects (font (size 1.27 1.27)) hide)
+    )

Commit message: production files
Parts:
- C501: value C_Small -> 100n
- R501: value 220R -> 22R
Changed lines of the file:
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@@
       (effects (font (size 1.27 1.27)) (justify right))
     )
-    (property "Value" "220R" (id 1) (at 93.98 31.7499 0)
+    (property "Value" "22R" (id 1) (at 93.98 31.7499 0)
       (effects (font (size 1.27 1.27)) (justify right))
     )
@@
     (in_bom yes) (on_board yes) (fields_autoplaced)
     (property "Reference" "C501" (id 0) (at 113.0363 33.02 90))
-    (property "Value" "C_Small" (id 1) (at 113.0363 35.56 90))
+    (property "Value" "100n" (id 1) (at 113.0363 35.56 90))
     (property "Footprint" "Capacitor_SMD:C_0603_1608Metric" (id 2) (at 113.03 39.37 0)
       (effects (font (size 1.27 1.27)) hide)
