File: inzynierka/_autosave-inzynierka.kicad_pcb (KiCad board)
At the start: 2 copper layers, 69.6 x 95.6 mm, 139 parts, among them J101 SHIELD_LEFT, J102 SHIELD_RIGHT, J104 PIEZO, J105 FPC, J106 FPC, Q501 SS8550, Q502 MMBT3904, SW101 DBG, T501 Transformer_Audio, U101 LM1117-3.3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

Commit message: production files
Parts:
- R204: value R_Small -> 51k
Connections:
- J106 pad MP: GND -> (no net)

Commit message: poprawione gerbery
Parts:
- SW101: footprint Button_Switch_SMD:SW_SPST_B3S-1000 -> Button_Switch_SMD:SW_SPST_TL3342
- moved SW101 0.50 mm to (88.0, 93.0)
Routing:
- net Net-(C112-Pad1): track 13.9 -> 12.6 mm
