File: pcb/inzynierka/transmiter.kicad_sch (KiCad schematic)
At the start: 12 parts, among them Q501 SS8550, Q502 MMBT3904, T501 Transformer_Audio

Commit message: progress before last consultation
Connections:
- net GND: now also D502.1 (K); no longer D502.2 (A)
- net at R503.2: now also D502.2 (A); no longer D502.1 (K)
Other:
- moved on the sheet: D502
Changed lines of the file:
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@@
     (pin "1")
   )
-  (symbol (lib_id "Device:LED_Small") (at 71.12 43.18 270) (unit 1)
+  (symbol (lib_id "Device:LED_Small") (at 71.12 43.18 90) (unit 1)
     (in_bom yes) (on_board yes) (fields_autoplaced)
-    (property "Reference" "D502" (id 0) (at 73.66 41.9734 90)
-      (effects (font (size 1.27 1.27)) (justify left))
+    (property "Reference" "D502" (id 0) (at 73.66 41.8464 90)
+      (effects (font (size 1.27 1.27)) (justify right))
     )
-    (property "Value" "BLUE" (id 1) (at 73.66 44.5134 90)
-      (effects (font (size 1.27 1.27)) (justify left))
+    (property "Value" "BLUE" (id 1) (at 73.66 44.3864 90)
+      (effects (font (size 1.27 1.27)) (justify right))
     )
     (property "Footprint" "LED_SMD:LED_0603_1608Metric" (id 2) (at 71.12 43.18 90)
