File: pcb/inzynierka/MIC_0.kicad_sch (KiCad schematic)
At the start: 20 parts, among them U202 MCP6L04x-xSL

Commit message: gotowa praca dyplomowa
Parts:
- C205, C207: value 117p -> 47p
- C209: value 39p -> 47p
- R202: value 25.5k -> 22k
- R204: value 51k -> 22k
Other:
- note added: "Third stage filter"
Changed lines of the file:
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@@
     (effects (font (size 3 3) italic) (justify left bottom))
   )
-  (text "Amplifier" (at 193.04 21.59 0)
+  (text "Third stage filter" (at 184.15 21.59 0)
     (effects (font (size 3 3) italic) (justify left bottom))
   )
@@
     (effects (font (size 3 3) italic) (justify left bottom))
   )
-  (text "Second stage filter" (at 130.81 21.59 0)
+  (text "Second stage filter" (at 125.73 21.59 0)
     (effects (font (size 3 3) italic) (justify left bottom))
   )
@@
     (in_bom yes) (on_board yes) (fields_autoplaced)
     (property "Reference" "C205" (id 0) (at 96.5263 24.13 90))
-    (property "Value" "117p" (id 1) (at 96.5263 26.67 90))
+    (property "Value" "47p" (id 1) (at 96.5263 26.67 90))
     (property "Footprint" "Capacitor_SMD:C_0603_1608Metric" (id 2) (at 96.52 30.48 0)
       (effects (font (size 1.27 1.27)) hide)
@@
     (in_bom yes) (on_board yes) (fields_autoplaced)
     (property "Reference" "R202" (id 0) (at 96.52 34.29 90))
-    (property "Value" "25.5k" (id 1) (at 96.52 36.83 90))
+    (property "Value" "22k" (id 1) (at 96.52 36.83 90))
     (property "Footprint" "Resistor_SMD:R_0603_1608Metric" (id 2) (at 96.52 40.64 0)
       (effects (font (size 1.27 1.27)) hide)
@@
     (in_bom yes) (on_board yes) (fields_autoplaced)
     (property "Reference" "C209" (id 0) (at 203.2063 24.13 90))
-    (property "Value" "39p" (id 1) (at 203.2063 26.67 90))
+    (property "Value" "47p" (id 1) (at 203.2063 26.67 90))
     (property "Footprint" "Capacitor_SMD:C_0603_1608Metric" (id 2) (at 203.2 30.48 0)
       (effects (font (size 1.27 1.27)) hide)
@@
     (in_bom yes) (on_board yes) (fields_autoplaced)
     (property "Reference" "R204" (id 0) (at 149.86 34.29 90))
-    (property "Value" "51k" (id 1) (at 149.86 36.83 90))
+    (property "Value" "22k" (id 1) (at 149.86 36.83 90))
     (property "Footprint" "Resistor_SMD:R_0603_1608Metric" (id 2) (at 149.86 40.64 0)
       (effects (font (size 1.27 1.27)) hide)
@@
     (in_bom yes) (on_board yes) (fields_autoplaced)
     (property "Reference" "C207" (id 0) (at 149.8663 24.13 90))
-    (property "Value" "117p" (id 1) (at 149.8663 26.67 90))
+    (property "Value" "47p" (id 1) (at 149.8663 26.67 90))
     (property "Footprint" "Capacitor_SMD:C_0603_1608Metric" (id 2) (at 149.86 30.48 0)
       (effects (font (size 1.27 1.27)) hide)
