File: pcb/inzynierka/inzynierka.kicad_sch (KiCad schematic)
At the start: 54 parts, among them J101 SHIELD_LEFT, J102 SHIELD_RIGHT, J104 PIEZO, J105 FPC, J106 FPC, SW101 DBG, U101 LM1117-3.3, U102 MCP6L04x-xSL, U103 LM239D, U201 SPU0410LR5H-QB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

Commit message: progress in thesis
Connections:
- net DBG_LED: now also D104.1 (K); no longer D104.2 (A)
- net GND: now also D101.1 (K), D102.1 (K); no longer D101.2 (A), D102.2 (A)
- net THRESHOLD_OP: now also D103.1 (K); no longer D103.2 (A)
- net at R110.2: now also D104.2 (A); no longer D104.1 (K)
- net at R107.2: now also D101.2 (A); no longer D101.1 (K)
- net at R108.2: now also D102.2 (A); no longer D102.1 (K)
- net at R109.2: now also D103.2 (A); no longer D103.1 (K)
Other:
- moved on the sheet: D101, D102, D103, D104
Changed lines of the file:
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@@
     (pin "1")
   )
-  (symbol (lib_id "Device:LED_Small") (at 142.24 43.18 270) (unit 1)
-    (in_bom yes) (on_board yes) (fields_autoplaced)
-    (property "Reference" "D101" (id 0) (at 144.78 41.9734 90)
-      (effects (font (size 1.27 1.27)) (justify left))
-    )
-    (property "Value" "5V" (id 1) (at 144.78 44.5134 90)
-      (effects (font (size 1.27 1.27)) (justify left))
+  (symbol (lib_id "Device:LED_Small") (at 142.24 43.18 90) (unit 1)
+    (in_bom yes) (on_board yes) (fields_autoplaced)
+    (property "Reference" "D101" (id 0) (at 144.78 41.8464 90)
+      (effects (font (size 1.27 1.27)) (justify right))
+    )
+    (property "Value" "5V" (id 1) (at 144.78 44.3864 90)
+      (effects (font (size 1.27 1.27)) (justify right))
     )
     (property "Footprint" "LED_SMD:LED_0603_1608Metric" (id 2) (at 142.24 43.18 90)
@@
     (pin "1")
   )
-  (symbol (lib_id "Device:LED_Small") (at 181.61 43.18 270) (unit 1)
-    (in_bom yes) (on_board yes) (fields_autoplaced)
-    (property "Reference" "D103" (id 0) (at 184.15 41.9734 90)
-      (effects (font (size 1.27 1.27)) (justify left))
-    )
-    (property "Value" "THOLD" (id 1) (at 184.15 44.5134 90)
-      (effects (font (size 1.27 1.27)) (justify left))
+  (symbol (lib_id "Device:LED_Small") (at 181.61 43.18 90) (unit 1)
+    (in_bom yes) (on_board yes) (fields_autoplaced)
+    (property "Reference" "D103" (id 0) (at 184.15 41.8464 90)
+      (effects (font (size 1.27 1.27)) (justify right))
+    )
+    (property "Value" "THOLD" (id 1) (at 184.15 44.3864 90)
+      (effects (font (size 1.27 1.27)) (justify right))
     )
     (property "Footprint" "LED_SMD:LED_0603_1608Metric" (id 2) (at 181.61 43.18 90)
@@
     (pin "1")
   )
-  (symbol (lib_id "Device:LED_Small") (at 165.1 43.18 270) (unit 1)
-    (in_bom yes) (on_board yes) (fields_autoplaced)
-    (property "Reference" "D104" (id 0) (at 167.64 41.9734 90)
-      (effects (font (size 1.27 1.27)) (justify left))
-    )
-    (property "Value" "DBG" (id 1) (at 167.64 44.5134 90)
-      (effects (font (size 1.27 1.27)) (justify left))
+  (symbol (lib_id "Device:LED_Small") (at 165.1 43.18 90) (unit 1)
+    (in_bom yes) (on_board yes) (fields_autoplaced)
+    (property "Reference" "D104" (id 0) (at 167.64 41.8464 90)
+      (effects (font (size 1.27 1.27)) (justify right))
+    )
+    (property "Value" "DBG" (id 1) (at 167.64 44.3864 90)
+      (effects (font (size 1.27 1.27)) (justify right))
     )
     (property "Footprint" "LED_SMD:LED_0603_1608Metric" (id 2) (at 165.1 43.18 90)
@@
     (pin "2")
   )
-  (symbol (lib_id "Device:LED_Small") (at 153.67 43.18 270) (unit 1)
-    (in_bom yes) (on_board yes) (fields_autoplaced)
-    (property "Reference" "D102" (id 0) (at 156.21 41.9734 90)
-      (effects (font (size 1.27 1.27)) (justify left))
-    )
-    (property "Value" "3V3" (id 1) (at 156.21 44.5134 90)
-      (effects (font (size 1.27 1.27)) (justify left))
+  (symbol (lib_id "Device:LED_Small") (at 153.67 43.18 90) (unit 1)
+    (in_bom yes) (on_board yes) (fields_autoplaced)
+    (property "Reference" "D102" (id 0) (at 156.21 41.8464 90)
+      (effects (font (size 1.27 1.27)) (justify right))
+    )
+    (property "Value" "3V3" (id 1) (at 156.21 44.3864 90)
+      (effects (font (size 1.27 1.27)) (justify right))
     )
     (property "Footprint" "LED_SMD:LED_0603_1608Metric" (id 2) (at 153.67 43.18 90)

Commit message: gotowa praca dyplomowa
Parts:
- R101, R102, R103: value 100k -> 4.7k
Other:
- moved on the sheet: H101, H102, H103, H104
